Commit message: Update darkie_maze_urdf.xacro

File: darkie_maze_urdf_description/urdf/darkie_maze_urdf.xacro (robot description, xacro)
@@ -405,3 +405,39 @@
   <child link="colorsensor_1"/>
 </joint>
+<ros2_control name="DynamixelSystem" type="system">
+  <hardware>
+    <plugin>dynamixel_hardware/DynamixelHardware</plugin>
+    <param name="device_name">/dev/ttyACM0</param>
+    <param name="baud_rate">1000000</param>
+  </hardware>
+  <!-- LEFT FRONT -->
+  <joint name="Revolute 18">
+    <command_interface name="velocity"/>
+    <state_interface name="velocity"/>
+    <state_interface name="position"/>
+  </joint>
+  <!-- RIGHT FRONT -->
+  <joint name="Revolute 17">
+    <command_interface name="velocity"/>
+    <state_interface name="velocity"/>
+    <state_interface name="position"/>
+  </joint>
+  <!-- LEFT REAR -->
+  <joint name=Revolute 19">
+    <command_interface name="velocity"/>
+    <state_interface name="velocity"/>
+    <state_interface name="position"/>
+  </joint>
+  <!-- RIGHT REAR -->
+  <joint name="Revolute 16">
+    <command_interface name="velocity"/>
+    <state_interface name="velocity"/>
+    <state_interface name="position"/>
+  </joint>
+<joint name="Revolute 20">
+    <command_interface name="position"/>
+    <state_interface name="velocity"/>
+    <state_interface name="position"/>
+  </joint>
+</ros2_control>
 </robot>

Commit message: Update darkie_maze_urdf.xacro

File: darkie_maze_urdf_description/urdf/darkie_maze_urdf.xacro (robot description, xacro)
@@ -424,5 +424,5 @@
   </joint>
   <!-- LEFT REAR -->
-  <joint name=Revolute 19">
+  <joint name="Revolute 19">
     <command_interface name="velocity"/>
     <state_interface name="velocity"/>

Commit message: Update darkie_maze_urdf.xacro

File: darkie_maze_urdf_description/urdf/darkie_maze_urdf.xacro (robot description, xacro)
@@ -324,5 +324,5 @@
   </collision>
 </link>
-<joint name="Revolute 7" type="continuous">
+<joint name="lidar_joint" type="continuous">
   <origin xyz="-0.031 -0.022 0.0072" rpy="0 0 0"/>
   <parent link="lidar_bottom_1"/>
@@ -340,5 +340,5 @@
   <child link="right_vl53lohsensor_1"/>
 </joint>
-<joint name="Revolute 16" type="continuous">
+<joint name="right_rear_wheel_joint" type="continuous">
   <origin xyz="0.052 -0.055 0.01125" rpy="0 0 0"/>
   <parent link="base_link"/>
@@ -346,5 +346,5 @@
   <axis xyz="1.0 0.0 0.0"/>
 </joint>
-<joint name="Revolute 17" type="continuous">
+<joint name="right_front_wheel_joint" type="continuous">
   <origin xyz="0.052 0.055 0.01125" rpy="0 0 0"/>
   <parent link="base_link"/>
@@ -352,5 +352,5 @@
   <axis xyz="-1.0 0.0 0.0"/>
 </joint>
-<joint name="Revolute 18" type="continuous">
+<joint name="left_front_wheel_joint" type="continuous">
   <origin xyz="-0.052 0.055 0.01125" rpy="0 0 0"/>
   <parent link="base_link"/>
@@ -358,5 +358,5 @@
   <axis xyz="-1.0 0.0 0.0"/>
 </joint>
-<joint name="Revolute 19" type="continuous">
+<joint name="left_rear_wheel_joint" type="continuous">
   <origin xyz="-0.052 -0.055 0.01125" rpy="0 0 0"/>
   <parent link="base_link"/>
@@ -364,5 +364,5 @@
   <axis xyz="1.0 0.0 0.0"/>
 </joint>
-<joint name="Revolute 20" type="continuous">
+<joint name="lidar_joint" type="continuous">
   <origin xyz="0.0 -0.075 0.0586" rpy="0 0 0"/>
   <parent link="base_link"/>
@@ -412,5 +412,5 @@
   </hardware>
   <!-- LEFT FRONT -->
-  <joint name="Revolute 18">
+  <joint name="left_front_wheel_joint">
     <command_interface name="velocity"/>
     <state_interface name="velocity"/>
@@ -418,5 +418,5 @@
   </joint>
   <!-- RIGHT FRONT -->
-  <joint name="Revolute 17">
+  <joint name="right_front_wheel_joint">
     <command_interface name="velocity"/>
     <state_interface name="velocity"/>
@@ -424,5 +424,5 @@
   </joint>
   <!-- LEFT REAR -->
-  <joint name="Revolute 19">
+  <joint name="left_rear_wheel_joint">
     <command_interface name="velocity"/>
     <state_interface name="velocity"/>
@@ -430,10 +430,10 @@
   </joint>
   <!-- RIGHT REAR -->
-  <joint name="Revolute 16">
+  <joint name="right_rear_wheel_joint">
     <command_interface name="velocity"/>
     <state_interface name="velocity"/>
     <state_interface name="position"/>
   </joint>
-<joint name="Revolute 20">
+<joint name="lidar_joint">
     <command_interface name="position"/>
     <state_interface name="velocity"/>

Commit message: Update darkie_maze_urdf.xacro

File: darkie_maze_urdf_description/urdf/darkie_maze_urdf.xacro (robot description, xacro)
@@ -411,29 +411,30 @@
     <param name="baud_rate">1000000</param>
   </hardware>
-  <!-- LEFT FRONT -->
   <joint name="left_front_wheel_joint">
+    <param name="id">1</param>
     <command_interface name="velocity"/>
+    <state_interface name="position"/>
     <state_interface name="velocity"/>
+  </joint>
+  <joint name="right_front_wheel_joint">
+    <param name="id">2</param>
+    <command_interface name="velocity"/>
     <state_interface name="position"/>
+    <state_interface name="velocity"/>
   </joint>
-  <!-- RIGHT FRONT -->
-  <joint name="right_front_wheel_joint">
+  <joint name="left_rear_wheel_joint">
+    <param name="id">3</param>
     <command_interface name="velocity"/>
+    <state_interface name="position"/>
     <state_interface name="velocity"/>
+  </joint>
+  <joint name="right_rear_wheel_joint">
+    <param name="id">4</param>
+    <command_interface name="velocity"/>
     <state_interface name="position"/>
-  </joint>
-  <!-- LEFT REAR -->
-  <joint name="left_rear_wheel_joint">
-    <command_interface name="velocity"/>
     <state_interface name="velocity"/>
-    <state_interface name="position"/>
-  </joint>
-  <!-- RIGHT REAR -->
-  <joint name="right_rear_wheel_joint">
-    <command_interface name="velocity"/>
-    <state_interface name="velocity"/>
-    <state_interface name="position"/>
   </joint>
 <joint name="lidar_joint">
+<param name="id">5</param>
     <command_interface name="position"/>
     <state_interface name="velocity"/>
